File: KiCAD-THT/WiFive55.sch (KiCad schematic (older format))
At the start: 54 parts, among them J2 Switched Output, J3 Breadboard, J4 Grounds, J5 555-esque, K1 FINDER-36.11, K1001 G5Q-1A, Q1 BS170, Q2 IRF540N, Q5 BC557, SW3 PRG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

Commit message: Space for Omron G3MB-202P
Parts:
- renumbered J4 to J1, J2 to J3, J3 to J8
Changed lines of the file:
@@
 $EndDescr
 $Comp
-L Connector_Generic:Conn_01x08 J3
+L Connector_Generic:Conn_01x08 J8
 U 1 1 5EE6EDC3
 P 1200 2300
-F 0 "J3" H 1150 2700 50  0000 L CNN
+F 0 "J8" H 1150 2700 50  0000 L CNN
 F 1 "Breadboard" V 1300 2100 50  0000 L CNN
 F 2 "Connector_PinHeader_2.54mm:PinHeader_1x08_P2.54mm_Horizontal" H 1200 2300 50  0001 C CNN
@@
 $EndComp
 $Comp
-L Connector:Screw_Terminal_01x03 J2
+L Connector:Screw_Terminal_01x03 J3
 U 1 1 5FF4F85F
 P 4600 2550
-F 0 "J2" V 4600 2300 50  0000 L CNN
+F 0 "J3" V 4600 2300 50  0000 L CNN
 F 1 "Switched Output" V 4700 2150 50  0000 L CNN
 F 2 "TerminalBlock:TerminalBlock_bornier-3_P5.08mm" H 4600 2550 50  0001 C CNN
@@
 	1400 1900 3200 1900
 $Comp
-L Connector_Generic:Conn_01x08 J4
+L Connector_Generic:Conn_01x08 J1
 U 1 1 60121331
 P 900 2300
-F 0 "J4" H 850 2700 50  0000 L CNN
+F 0 "J1" H 850 2700 50  0000 L CNN
 F 1 "Grounds" V 1000 2150 50  0000 L CNN
 F 2 "Connector_PinHeader_2.54mm:PinHeader_1x08_P2.54mm_Vertical" H 900 2300 50  0001 C CNN

Commit message: update silks
Parts:
- R4: value 200 -> 470
Other:
- note added: "GPIO0 !PROG/!BTN\nGPIO1 TX/!LED\nGPIO2 !OUTPUT\nGPIO3 RX\n*R9 to suit output device. E.g. zero ohms"
- note removed: "GPIO0 !PROG/!BTN\nGPIO1 TX/!LED\nGPIO2 !OUTPUT\nGPIO3 RX"
- moved on the sheet: H2
Changed lines of the file:
@@
 Wire Wire Line
 	1400 2600 2150 2600
-Text Notes 3600 4450 0    50   ~ 0
-GPIO0 !PROG/!BTN\nGPIO1 TX/!LED\nGPIO2 !OUTPUT\nGPIO3 RX
+Text Notes 3600 4550 0    50   ~ 0
+GPIO0 !PROG/!BTN\nGPIO1 TX/!LED\nGPIO2 !OUTPUT\nGPIO3 RX\n*R9 to suit output device. E.g. zero ohms
 Wire Wire Line
 	2450 2500 2450 2950
@@
 L Mechanical:MountingHole H2
 U 1 1 605643E9
-P 3500 4000
-F 0 "H2" V 3500 3800 50  0000 L CNN
-F 1 "MountingHole" V 3650 3700 50  0000 L CNN
-F 2 "MountingHole:MountingHole_3.2mm_M3" H 3500 4000 50  0001 C CNN
-F 3 "~" H 3500 4000 50  0001 C CNN
-	1    3500 4000
+P 3500 3850
+F 0 "H2" V 3500 3650 50  0000 L CNN
+F 1 "MountingHole" V 3650 3550 50  0000 L CNN
+F 2 "MountingHole:MountingHole_3.2mm_M3" H 3500 3850 50  0001 C CNN
+F 3 "~" H 3500 3850 50  0001 C CNN
+	1    3500 3850
 	0    -1   -1   0
 $EndComp
@@
 P 4700 1300
 F 0 "R4" V 4700 1200 50  0000 L CNN
-F 1 "200" H 4650 1500 50  0000 L CNN
+F 1 "470" H 4650 1500 50  0000 L CNN
 F 2 "Resistor_THT:R_Axial_DIN0204_L3.6mm_D1.6mm_P2.54mm_Vertical" V 4630 1300 50  0001 C CNN
 F 3 "~" H 4700 1300 50  0001 C CNN
